File: prod-files/K-Logic-Devboard.kicad_pcb (KiCad board)
At the start: 2 copper layers, 21 x 51 mm, 35 parts, among them J1 USB_C_Receptacle_USB2.0_14P, J2 Conn_01x20, J3 Conn_01x20, J4 Conn_01x03, SW1 SW_Push, U1 RP2040, U2 MCP1700x-330xxTT, U3 W25Q16JVZPIQ TR, Y1 12 Mhz

Commit message: we done
Routing:
- removed copper zone on B.Cu, net GND
Changed lines of the file:
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@@
 		(net 2)
 		(net_name "GND")
-		(layers "F.Cu" "B.Cu")
+		(layer "F.Cu")
 		(hatch edge 0.5)
 		(priority 1)
